File: output/pcbs/fiano.kicad_pcb (KiCad board)
At the start: 2 copper layers, 195.4 x 160 mm, 51 parts

Commit message: modified pcb
Parts:
- added _1: , MountingHole_2.2mm_M2_Pad_Via, F.Cu at (140.0, 15.0)
- added _2: , MountingHole_2.2mm_M2_Pad_Via, F.Cu at (100.0, 60.0)
- added _3: , MountingHole_2.2mm_M2_Pad_Via, F.Cu at (140.0, 95.0)
- added _4: , MountingHole_2.2mm_M2_Pad_Via, F.Cu at (260.2, 140.5)
- added _5: , MountingHole_2.2mm_M2_Pad_Via, F.Cu at (214.9, 76.5)
- moved MCU1 166.7 mm to (160.0, 90.5), turned to 90 degrees
- moved D22 141.4 mm to (258.4, 127.2)
- moved D1 141.4 mm to (100.0, 85.0)
- moved D10 141.4 mm to (160.0, 30.0)
- moved D11 141.4 mm to (180.0, 95.0)
- moved D12 141.4 mm to (180.0, 75.0)
- moved D13 141.4 mm to (180.0, 55.0)
- moved D14 141.4 mm to (180.0, 35.0)
- moved D15 141.4 mm to (200.0, 100.0)
- moved D16 141.4 mm to (200.0, 80.0)
- moved D17 141.4 mm to (200.0, 60.0)
- moved D18 141.4 mm to (200.0, 40.0)
- moved D19 141.4 mm to (247.9, 149.1)
- moved D2 141.4 mm to (120.0, 95.0)
- moved D20 141.4 mm to (236.2, 131.6)
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Connections:
- B1 pad 2: reset -> RST
Routing:
- net GND: track 263.7 -> 0.00 mm
- net P3: track 235.1 -> 0.00 mm
- net P9: track 233.2 -> 0.00 mm
- net P8: track 154.8 -> 0.00 mm
- net VCC: track 116.1 -> 0.00 mm
- net P18: track 87.5 -> 0.00 mm
- net P15: track 79.1 -> 20.0 mm
- net P14: track 57.5 -> 0.00 mm
- net index_hometop: track 0.00 -> 31.5 mm
- net inner_hometop: track 0.00 -> 31.3 mm
- net inner_home: track 0.00 -> 31.2 mm
- net inner_top: track 0.00 -> 31.2 mm
- net inner_2: track 28.0 -> 0.00 mm
- net outer_2: track 27.5 -> 0.00 mm
- net outer_3: track 27.2 -> 0.00 mm
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
Commit message: wired pcb
Parts:
- removed OLED1: OLED, lib:OLED_headers
- removed _1, _2, _3, _4, _5: , MountingHole_2.2mm_M2_Pad_Via
- added B2: , E73:SW_TACT_ALPS_SKQGABE010, F.Cu at (400.0, 65.0)
- added D25: , ComboDiode, F.Cu at (420.0, 125.0)
- added D26: , ComboDiode, F.Cu at (420.0, 105.0)
- added D27: , ComboDiode, F.Cu at (400.0, 130.0)
- added D28: , ComboDiode, F.Cu at (400.0, 110.0)
- added D29: , ComboDiode, F.Cu at (400.0, 90.0)
- added D30: , ComboDiode, F.Cu at (380.0, 120.0)
- added D31: , ComboDiode, F.Cu at (380.0, 100.0)
- added D32: , ComboDiode, F.Cu at (380.0, 80.0)
- added D33: , ComboDiode, F.Cu at (360.0, 125.0)
- added D34: , ComboDiode, F.Cu at (360.0, 105.0)
- added D35: , ComboDiode, F.Cu at (360.0, 85.0)
- added D36: , ComboDiode, F.Cu at (340.0, 150.0)
- added D37: , ComboDiode, F.Cu at (340.0, 130.0)
- added D38: , ComboDiode, F.Cu at (340.0, 110.0)
- added D39: , ComboDiode, F.Cu at (340.0, 90.0)
- added D40: , ComboDiode, F.Cu at (292.1, 199.1)
- added D41: , ComboDiode, F.Cu at (303.8, 181.6)
- added D42: , ComboDiode, F.Cu at (317.0, 165.2)
- added D43: , ComboDiode, F.Cu at (281.6, 177.2)
- added D44: , ComboDiode, F.Cu at (293.6, 160.0)
- added MCU2: , ProMicro, F.Cu at (380.0, 74.0)
- added S25: , MX, F.Cu at (420.0, 120.0)
- added S26: , MX, F.Cu at (420.0, 100.0)
- added S27: , MX, F.Cu at (400.0, 125.0)
- added S28: , MX, F.Cu at (400.0, 105.0)
- added S29: , MX, F.Cu at (400.0, 85.0)
- added S30: , MX, F.Cu at (380.0, 115.0)
- added S31: , MX, F.Cu at (380.0, 95.0)
- added S32: , MX, F.Cu at (380.0, 75.0)
- added S33: , MX, F.Cu at (360.0, 120.0)
- added S34: , MX, F.Cu at (360.0, 100.0)
- added S35: , MX, F.Cu at (360.0, 80.0)
- added S36: , MX, F.Cu at (340.0, 145.0)
- added S37: , MX, F.Cu at (340.0, 125.0)
- added S38: , MX, F.Cu at (340.0, 105.0)
- added S39: , MX, F.Cu at (340.0, 85.0)
- added S40: , MX, F.Cu at (295.0, 195.0)
- added S41: , MX, F.Cu at (307.0, 177.8)
- added S42: , MX, F.Cu at (320.5, 161.7)
- added S43: , MX, F.Cu at (284.6, 173.2)
- added S44: , MX, F.Cu at (296.9, 156.2)
- added TRRS1: TRRS-PJ-320A-dual, TRRS-PJ-320A-dual, F.Cu at (184.0, 124.4)
- added TRRS2: TRRS-PJ-320A-dual, TRRS-PJ-320A-dual, F.Cu at (306.0, 124.4)
- moved S23 198.4 mm to (440.0, 130.0), turned to 0 degrees
- moved S24 197.1 mm to (420.0, 140.0), turned to 0 degrees
- moved D23 195.2 mm to (440.0, 135.0), turned to 0 degrees
- moved D24 194.0 mm to (420.0, 145.0), turned to 0 degrees
- moved S18 160.1 mm to (195.0, 195.0), turned to 35 degrees
- moved D18 159.1 mm to (197.9, 199.1), turned to 35 degrees
- moved D14 118.8 mm to (150.0, 150.0)
- moved S14 118.8 mm to (150.0, 145.0)
- moved S20 72.0 mm to (169.5, 161.7), turned to 45 degrees
- moved D20 71.6 mm to (173.0, 165.2), turned to 45 degrees
- moved D1 70.7 mm to (50.0, 135.0)
- moved D10 70.7 mm to (110.0, 80.0)
- moved D2 70.7 mm to (70.0, 145.0)
- moved D3 70.7 mm to (70.0, 125.0)
- moved D4 70.7 mm to (70.0, 105.0)
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Connections:
- net GND renamed GNDL
- net P4 renamed L4
- net P5 renamed L5
- net P6 renamed L6
- net P7 renamed L7
- net RAW renamed RAWL
- net RST renamed RSTL
- net outer_3 renamed mirror_pinky_bottom
- D1 pad 1: P8 -> L8
- D10 pad 1: P21 -> L21
- D11 pad 1: P18 -> L19
- D11 pad 2: index_bottom -> index_home
- D12 pad 1: P19 -> L20
- D12 pad 2: index_home -> index_hometop
- D13 pad 1: P20 -> L21
- D13 pad 2: index_hometop -> index_top
- D14 pad 1: P21 -> L18
- D14 pad 2: index_top -> inner_bottom
- D15 pad 1: P18 -> L19
- D15 pad 2: inner_bottom -> inner_home
- D16 pad 1: P19 -> L20
- D16 pad 2: inner_home -> inner_hometop
- D17 pad 1: P20 -> L21
- D17 pad 2: inner_hometop -> inner_top
- D18 pad 1: P21 -> L8
- D18 pad 2: inner_top -> inner_1
- D19 pad 1: (no net) -> L8
- D19 pad 2: inner_1 -> inner_2
- D2 pad 1: P19 -> L19
- D20 pad 1: (no net) -> L8
- D20 pad 2: inner_2 -> inner_3
- D21 pad 1: (no net) -> L18
- D21 pad 2: inner_3 -> outer_1
- D22 pad 1: (no net) -> L18
- D22 pad 2: outer_1 -> outer_2
- D23 pad 1: (no net) -> R8
- D23 pad 2: outer_2 -> mirror_prepinky_home
- D24 pad 1: (no net) -> R19
- D3 pad 1: P20 -> L20
- D4 pad 1: P21 -> L21
- D5 pad 1: P19 -> L19
- D6 pad 1: P20 -> L20
- D7 pad 1: P21 -> L21
- D8 pad 1: P19 -> L19
- D9 pad 1: P20 -> L20
- MCU1 pad 10: P14 -> L14
- MCU1 pad 11: P16 -> L16
- MCU1 pad 12: P10 -> L10
- MCU1 pad 13: P1 -> L1
- MCU1 pad 14: P0 -> L0
- MCU1 pad 17: P2 -> L2
- MCU1 pad 18: P3 -> L3
- MCU1 pad 23: P8 -> L8
- MCU1 pad 24: P9 -> L9
- MCU1 pad 4: VCC -> VCCL
- MCU1 pad 5: P21 -> L21
- MCU1 pad 6: P20 -> L20
- MCU1 pad 7: P19 -> L19
- MCU1 pad 8: P18 -> L18
- MCU1 pad 9: P15 -> L15
- S1 pad 1: P9 -> L9
- S10 pad 1: P14 -> L14
- S11 pad 1: P9 -> L15
- S11 pad 2: index_bottom -> index_home
- S12 pad 1: P15 -> L15
- S12 pad 2: index_home -> index_hometop
- S13 pad 1: P15 -> L15
- S13 pad 2: index_hometop -> index_top
- S14 pad 1: P15 -> L10
- S14 pad 2: index_top -> inner_bottom
- S15 pad 1: P10 -> L16
- S15 pad 2: inner_bottom -> inner_home
- S16 pad 1: P16 -> L16
- S16 pad 2: inner_home -> inner_hometop
- S17 pad 1: P16 -> L16
- S17 pad 2: inner_hometop -> inner_top
- S18 pad 1: P16 -> L16
- S18 pad 2: inner_top -> inner_1
- S19 pad 1: P16 -> L15
- S19 pad 2: inner_1 -> inner_2
- S2 pad 1: P9 -> L9
- S20 pad 1: P15 -> L14
- S20 pad 2: inner_2 -> inner_3
- S21 pad 1: P14 -> L16
- S21 pad 2: inner_3 -> outer_1
- S22 pad 1: P16 -> L15
- S22 pad 2: outer_1 -> outer_2
- S23 pad 1: P15 -> R9
- S23 pad 2: outer_2 -> mirror_prepinky_home
- S24 pad 1: P14 -> R9
- S3 pad 1: P9 -> L9
- S4 pad 1: P9 -> L9
- S5 pad 1: P10 -> L10
- S6 pad 1: P10 -> L10
- S7 pad 1: P10 -> L10
- S8 pad 1: P14 -> L14
- S9 pad 1: P14 -> L14
Routing:
- net L15: track 0.00 -> 437.4 mm
- net L8: track 0.00 -> 308.4 mm
- net R8: track 0.00 -> 299.2 mm
- net R16: track 0.00 -> 245.2 mm
- net L19: track 0.00 -> 228.9 mm
- net L16: track 0.00 -> 211.6 mm
- net L18: track 0.00 -> 203.0 mm
- net R18: track 0.00 -> 176.1 mm
- net R19: track 0.00 -> 168.6 mm
- net R15: track 0.00 -> 156.2 mm
- net R14: track 0.00 -> 151.0 mm
- net R10: track 0.00 -> 149.8 mm
- net GNDR: track 0.00 -> 143.3 mm
- net L20: track 0.00 -> 143.3 mm
- net R20: track 0.00 -> 143.2 mm
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Other:
- board size 195.4 x 160 mm -> 430 x 160 mm
